File: LightingUPSEagle/LightingUPS-Sensor_v1.brd (EAGLE design)
At the start: 84 x 102 mm, 4 parts

Commit message: Add files via upload
Parts:
- removed J1: (no value), SparkFun-Connectors:1X02
- moved J2 23.3 mm to (62.2, 8.89)
- moved U$5 0.22 mm to (8.89, 18.0)
Connections:
- net N$1: no longer J1.2
- net N$2: no longer J1.1
Routing:
- net N$3: track 47.0 -> 77.5 mm
- net N$2: track 17.1 -> 0.00 mm
- net N$1: track 12.0 -> 0.00 mm
Other:
- outline, holes or cut-outs redrawn
- board text added: "The corresponding holes in the box are to be located 18mm down from the top edge"
- board text removed: "Holes in box are to be located 18mm down from the top edge"
Changed lines of the file:
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@@
 <plain>
 <wire x1="0" y1="0" x2="84" y2="0" width="0" layer="20"/>
-<wire x1="84" y1="0" x2="84" y2="36" width="0" layer="20"/>
+<wire x1="84" y1="0" x2="84" y2="11" width="0" layer="20"/>
+<wire x1="84" y1="25" x2="84" y2="36" width="0" layer="20"/>
 <wire x1="84" y1="36" x2="0" y2="36" width="0" layer="20"/>
 <wire x1="0" y1="36" x2="0" y2="0" width="0" layer="20"/>
-<text x="77.47" y="23.495" size="1.4224" layer="21" font="vector" rot="R270">Photocell</text>
-<text x="44.45" y="3.81" size="1.4224" layer="21" font="vector">Lighting UPS Sensor
+<text x="91.44" y="22.225" size="1.4224" layer="21" font="vector" rot="R270">Photocell</text>
+<text x="43.18" y="1.27" size="1.4224" layer="21" font="vector">Lighting UPS Sensor
 V1.0 May 2017</text>
 <hole x="3.2" y="32.8" drill="3.2"/>
@@
 <text x="24.765" y="16.51" size="1.4224" layer="21" font="vector">Motion
 Detector</text>
-<text x="38.1" y="13.335" size="1.6764" layer="21" font="vector">En
+<text x="43.18" y="13.335" size="1.6764" layer="21" font="vector">En
 Out
 Vcc
@@
 <hole x="61.8" y="93" drill="1.4"/>
 <dimension x1="49.53" y1="93" x2="49.53" y2="80" x3="57.15" y3="86.5" textsize="1.778" layer="1"/>
-<text x="10.16" y="87.63" size="1.4224" layer="21" font="vector">Holes in box are to be
+<text x="10.16" y="87.63" size="1.4224" layer="21" font="vector">The corresponding holes
+in the box are to be
 located 18mm down from
 the top edge</text>
+<wire x1="70" y1="11" x2="84" y2="11" width="0.254" layer="20"/>
+<wire x1="84" y1="11" x2="84" y2="25" width="0.1" layer="20"/>
+<wire x1="84" y1="25" x2="70" y2="25" width="0.254" layer="20"/>
+<wire x1="70" y1="25" x2="70" y2="11" width="0.254" layer="20"/>
+<dimension x1="70" y1="11" x2="84" y2="11" x3="77" y3="2.54" textsize="1.778" layer="20"/>
+<hole x="73" y="22" drill="2"/>
+<hole x="73" y="14" drill="2"/>
+<hole x="77" y="19.8" drill="1.6"/>
+<hole x="77" y="16.2" drill="1.6"/>
+<dimension x1="73" y1="13.97" x2="77" y2="13.97" x3="75" y3="7.62" textsize="1.778" layer="20"/>
+<dimension x1="65" y1="18" x2="65" y2="14" x3="67.31" y3="16" textsize="1.778" layer="20" width="0.1" extlength="4"/>
+<dimension x1="77.47" y1="18" x2="77.47" y2="16.2" x3="87.63" y3="17.1" textsize="1.778" layer="20"/>
+<dimension x1="32.8" y1="-7.62" x2="73" y2="-7.62" x3="52.9" y3="-4.96099375" textsize="1.778" layer="20"/>
+<dimension x1="41.91" y1="14" x2="41.91" y2="3.2" x3="39.37" y3="8.6" textsize="1.778" layer="20"/>
+<circle x="77" y="18" radius="2.5" width="0.1" layer="20"/>
 </plain>
 <attributes>
@@
 </autorouter>
 <elements>
-<element name="J1" library="SparkFun-Connectors" package="1X02" value="" x="76.42" y="17.78" smashed="yes" rot="R180">
-<attribute name="NAME" x="70.4088" y="19.3462" size="1.27" layer="25" ratio="10" rot="R270"/>
-<attribute name="VALUE" x="77.69" y="20.955" size="1.27" layer="27" rot="R180"/>
-</element>
-<element name="U$5" library="special-drill" package="DRILL_0.2500" value="" x="8.89" y="17.78"/>
+<element name="U$5" library="special-drill" package="DRILL_0.2500" value="" x="8.89" y="18"/>
 <element name="U$1" library="special-drill" package="DRILL_0.2500" value="" x="24.8875" y="26.475"/>
-<element name="J2" library="SparkFun-Connectors" package="1X02" value="" x="71.12" y="30.48" rot="R270"/>
+<element name="J2" library="SparkFun-Connectors" package="1X02" value="" x="62.23" y="8.89" rot="R270"/>
 </elements>
 <signals>
 <signal name="N$1">
-<contactref element="J1" pad="2"/>
 <contactref element="J2" pad="2"/>
-<wire x1="73.88" y1="17.78" x2="73.88" y2="26.45" width="0.4064" layer="16"/>
-<wire x1="73.88" y1="26.45" x2="72.39" y2="27.94" width="0.4064" layer="16"/>
-<wire x1="72.39" y1="27.94" x2="71.12" y2="27.94" width="0.4064" layer="16"/>
 </signal>
 <signal name="N$2">
-<contactref element="J1" pad="1"/>
 <contactref element="J2" pad="1"/>
-<wire x1="76.42" y1="17.78" x2="76.42" y2="28.99" width="0.4064" layer="16"/>
-<wire x1="76.42" y1="28.99" x2="74.93" y2="30.48" width="0.4064" layer="16"/>
-<wire x1="74.93" y1="30.48" x2="71.12" y2="30.48" width="0.4064" layer="16"/>
 </signal>
 <signal name="N$3">
-<wire x1="18" y1="74.93" x2="18" y2="27.94" width="0.254" layer="1" style="shortdash"/>
+<wire x1="18" y1="74.93" x2="18" y2="-2.54" width="0.254" layer="1" style="shortdash"/>
 </signal>
 <signal name="N$4">

Commit message: Add files via upload
Parts:
- removed J2: (no value), SparkFun-Connectors:1X02
- added J1: (no value), SparkFun-Connectors:1X04
- added J3: (no value), SparkFun-Connectors:2X3-SHROUDED
- added R1: PHOTOCELLPTH, SparkFun-Sensors:PHOTOCELL
- moved U$1 1.89 mm to (23.0, 26.5)
Connections:
- new net N$5: J1.4, J3.1
- new net N$6: J1.3, J3.3
- new net N$7: J1.2, J3.5
- new net N$8: J1.1, J3.6
- net N$1: now also J3.4, R1.1; no longer J2.2
- net N$2: now also J3.2, R1.2; no longer J2.1
Routing:
- net N$5: track 0.00 -> 44.6 mm
- net N$4: track 44.0 -> 0.00 mm
- net N$3: track 77.5 -> 35.6 mm
- net N$6: track 0.00 -> 34.4 mm
- net N$2: track 0.00 -> 25.6 mm
- net N$1: track 0.00 -> 24.4 mm
- net N$7: track 0.00 -> 24.3 mm
- net N$8: track 0.00 -> 16.9 mm
Other:
- board size 84 x 102 mm -> 113.2 x 113 mm
- board text added: "Gnd Vcc Out En"
- board text removed: "En Out Vcc Gnd"
