File: LightingUPSEagle/LightingUPS-SensorAssembly_v1.brd (EAGLE design)
At the start: 84 x 36 mm, 5 parts

Commit message: Add files via upload
Routing:
- net N$3: track 0.00 -> 35.6 mm
Other:
- board size 84 x 36 mm -> 113.2 x 113 mm
- board text added: "Box center line"
- board text added: "The corresponding holes in the box are to be located 17.5mm down from the top edge"
Changed lines of the file:
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@@
 Out
 En</text>
+<hole x="44.8" y="43.23" drill="2"/>
+<hole x="61.8" y="43.23" drill="2"/>
+<wire x1="39.8" y1="38.63" x2="39.8" y2="89.43" width="0.254" layer="20"/>
+<wire x1="39.8" y1="89.43" x2="66.8" y2="89.43" width="0.6096" layer="20"/>
+<wire x1="66.8" y1="89.43" x2="66.8" y2="38.63" width="0.254" layer="20"/>
+<wire x1="66.8" y1="38.63" x2="39.8" y2="38.63" width="0.254" layer="20"/>
+<dimension x1="39.37" y1="38.63" x2="39.37" y2="89.43" x3="64.77" y3="64.03" textsize="1.778" layer="1"/>
+<dimension x1="39.8" y1="90.17" x2="66.8" y2="90.17" x3="53.3" y3="85.09" textsize="1.778" layer="1"/>
+<text x="16.51" y="52.07" size="1.4224" layer="21" font="vector" rot="R90">Box center line</text>
+<dimension x1="18" y1="74.93" x2="39.8" y2="74.93" x3="28.9" y3="73.66" textsize="1.778" layer="1"/>
+<dimension x1="57.15" y1="38.63" x2="57.15" y2="43.23" x3="58.42" y3="40.93" textsize="1.778" layer="1"/>
+<dimension x1="18" y1="46.99" x2="44.8" y2="46.99" x3="31.4" y3="49.530003125" textsize="1.778" layer="1"/>
+<dimension x1="39.8" y1="48.26" x2="44.8" y2="48.26" x3="42.3" y3="46.99" textsize="1.778" layer="1"/>
+<dimension x1="44.8" y1="53.34" x2="61.8" y2="53.34" x3="53.3" y3="52.07" textsize="1.778" layer="1"/>
+<dimension x1="73.66" y1="91" x2="73.66" y2="113" x3="71.12" y3="102" textsize="1.778" layer="1"/>
+<hole x="44.8" y="104" drill="2.77"/>
+<hole x="61.8" y="104" drill="2.77"/>
+<dimension x1="49.53" y1="104" x2="49.53" y2="91" x3="57.15" y3="97.5" textsize="1.778" layer="1"/>
+<text x="10.16" y="99.06" size="1.4224" layer="21" font="vector">The corresponding holes
+in the box are to be
+located 17.5mm down from
+the top edge</text>
 <hole x="81" y="22" drill="2.8"/>
 <hole x="73" y="14" drill="2.8"/>
+<hole x="106.21" y="19.8" drill="2"/>
+<hole x="106.21" y="16.2" drill="2"/>
+<dimension x1="106.68" y1="19.8" x2="106.68" y2="16.2" x3="116.84" y3="18" textsize="1.778" layer="20"/>
+<hole x="18" y="78" drill="4.4"/>
+<hole x="114.75" y="78" drill="4.4"/>
+<wire x1="113.21" y1="25" x2="113.18" y2="25" width="0.254" layer="20"/>
+<wire x1="113.18" y1="25" x2="99.21" y2="25" width="0.254" layer="20"/>
+<wire x1="99.21" y1="11" x2="113.18" y2="11" width="0.254" layer="20"/>
+<wire x1="113.18" y1="11" x2="113.21" y2="11" width="0.254" layer="20"/>
+<wire x1="99.21" y1="25" x2="99.21" y2="11" width="0.254" layer="20"/>
+<wire x1="113.18" y1="25" x2="113.18" y2="11" width="0.254" layer="20"/>
+<dimension x1="99.21" y1="9.73" x2="113.21" y2="9.73" x3="106.21" y3="6.35" textsize="1.778" layer="20"/>
+<dimension x1="91.67" y1="22" x2="91.67" y2="14" x3="93.98" y3="18" textsize="1.778" layer="20" width="0.1" extlength="4"/>
+<hole x="110.21" y="22" drill="2"/>
+<hole x="102.21" y="14" drill="2"/>
+<dimension x1="102.21" y1="24.13" x2="106.21" y2="24.13" x3="104.21" y3="30.48" textsize="1.778" layer="20"/>
 <hole x="44.8" y="31.7" drill="3.2"/>
 <hole x="61.8" y="31.8" drill="3.2"/>
+<wire x1="39.8" y1="91" x2="66.8" y2="91" width="0.6096" layer="20"/>
+<wire x1="66.8" y1="91" x2="66.8" y2="113" width="0.254" layer="20"/>
+<wire x1="66.8" y1="113" x2="39.8" y2="113" width="0.254" layer="20"/>
+<wire x1="39.8" y1="113" x2="39.8" y2="91" width="0.254" layer="20"/>
+<hole x="114.75" y="-18.75" drill="4.4"/>
+<hole x="-78.75" y="-18.75" drill="4.4"/>
+<hole x="-78.75" y="78" drill="4.4"/>
 <circle x="18" y="18" radius="3.175" width="0.254" layer="21"/>
 </plain>
@@
 <element name="U$1" library="special-drill" package="DRILL_0.2500" value="" x="23" y="26.475"/>
 <element name="R1" library="SparkFun-Sensors" package="PHOTOCELL" value="PHOTOCELLPTH" x="77" y="18" smashed="yes" rot="R270">
-<attribute name="NAME" x="73.4" y="21" size="0.8128" layer="25" rot="R270"/>
+<attribute name="NAME" x="79.4" y="20" size="0.8128" layer="25" rot="R270"/>
 <attribute name="VALUE" x="76.54" y="31.43" size="0.8128" layer="27" rot="R270"/>
 </element>
 <element name="J1" library="SparkFun-Connectors" package="1X04" value="" x="46" y="14.2" smashed="yes" rot="R90">
 <attribute name="PROD_ID" value="CONN-09696" x="46" y="14.2" size="1.778" layer="27" rot="R90" display="off"/>
-<attribute name="NAME" x="46.8362" y="25.4212" size="1.27" layer="25" ratio="10" rot="R180"/>
+<attribute name="NAME" x="46.8362" y="12.4212" size="1.27" layer="25" ratio="10" rot="R180"/>
 <attribute name="VALUE" x="49.175" y="12.93" size="1.27" layer="27" rot="R90"/>
 </element>
@@
 </elements>
 <signals>
+<signal name="N$3">
+<wire x1="18" y1="74.93" x2="18" y2="39.37" width="0.254" layer="1" style="shortdash"/>
+</signal>
 <signal name="N$1">
 <contactref element="J3" pad="4"/>
