File: LightingUPSEagle/LightingUPS-AC_v4.brd (EAGLE design)
At the start: 113.2 x 113 mm, 5 parts

Commit message: Add files via upload
Parts:
- removed U$5: (no value), special-drill:DRILL_0.2500
- added D1: (no value), SparkFun-DiscreteSemi:DIODE-1N4001
- added J2: (no value), SparkFun-Connectors:1X02
- added J4, J5: (no value), SparkFun-Connectors:1X01
- added K1: JS1-5V, relay:JS-M
- added OK1: SFH620A, optocoupler:DIL04
- added R2: 220K, SparkFun-Passives:AXIAL-0.4
- added U$2, U$3, U$4: (no value), SparkFun-Electromechanical:STAND-OFF
- added X1, X2, X3: (no value), con-wago-500:W237-102
- J1: device SparkFun-Connectors:1X04 -> SparkFun-Connectors:1X02
- J3: device SparkFun-Connectors:2X3-SHROUDED -> SparkFun-Connectors:1X01
- R1: value PHOTOCELLPTH -> 220K; device SparkFun-Sensors:PHOTOCELL -> SparkFun-Passives:AXIAL-0.4
- U$1: device special-drill:DRILL_0.2500 -> SparkFun-Electromechanical:STAND-OFF
- moved R1 65.5 mm to (16.5, 43.2), turned to 0 degrees
- moved U$1 38.2 mm to (3.81, 41.9)
- moved J3 32.9 mm to (30.5, 24.1), flipped to the top, turned to 0 degrees
- moved J1 26.8 mm to (36.8, 39.4)
Connections:
- removed net N$7: J1.2, J3.5
- new net N$11: R2.P$1, X1.1, X2.2, X3.2
- new net N$12: J5.1, K1.NO, R1.P$1, X1.2
- new net N$3: J3.1, K1.C, X2.1
- new net N$4: D1.A, J2.1, K1.2
- new net N$9: OK1.1, R1.P$2
- net N$1: now also J4.1, X3.1; no longer J3.4, R1.1
- net N$2: now also J1.1, OK1.3; no longer J3.2, R1.2
- net N$5: now also D1.C, J2.2, K1.1; no longer J1.4, J3.1
- net N$6: now also J1.2, OK1.4; no longer J1.3, J3.3
- net N$8: now also OK1.2, R2.P$2; no longer J1.1, J3.6
Routing:
- net N$11: track 0.00 -> 62.1 mm
- net N$12: track 0.00 -> 51.0 mm
- net N$6: track 34.4 -> 3.81 mm
- net N$7: track 24.3 -> 0.00 mm
- net N$2: track 25.6 -> 3.81 mm
- net N$4: track 0.00 -> 20.2 mm
- net N$1: track 24.4 -> 7.64 mm
- net N$8: track 16.9 -> 4.34 mm
- net N$3: track 35.6 -> 26.9 mm
- net N$5: track 44.6 -> 49.6 mm
- net N$9: track 0.00 -> 4.34 mm
Other:
- board size 113.2 x 113 mm -> 47.3 x 45.7 mm
- board text added: "+"
- board text added: "JS1-5V"
- board text added: "Lighting UPS AC V4.0 Dec 2016"
- board text added: "Mains"
- board text added: "Mains Detect"
- board text added: "Relay Coil"
- board text added: "To AC Adapter"
- board text added: "To Battery Charger"
- board text removed: "Box center line"
- board text removed: "Gnd Vcc Out En"
- board text removed: "Lighting UPS Sensor V1.1 June 2017"
- board text removed: "Motion Detector"
- board text removed: "Photocell"
- board text removed: "The corresponding holes in the box are to be located 17.5mm down from the top edge"
