File: LightingUPSEagle/LightingUPS-BatteryTray_v1.brd (EAGLE design)
At the start: 113.2 x 113 mm, 5 parts

Commit message: Add files via upload
Parts:
- removed J1: (no value), SparkFun-Connectors:1X04
- removed J3: (no value), SparkFun-Connectors:2X3-SHROUDED
- removed R1: PHOTOCELLPTH, SparkFun-Sensors:PHOTOCELL
- removed U$1, U$5: (no value), special-drill:DRILL_0.2500
Connections:
- removed net N$1: J3.4, R1.1
- removed net N$2: J3.2, R1.2
- removed net N$5: J1.4, J3.1
- removed net N$6: J1.3, J3.3
- removed net N$7: J1.2, J3.5
- removed net N$8: J1.1, J3.6
Routing:
- net N$1: track 24.4 -> 137.0 mm
- net N$5: track 44.6 -> 0.00 mm
- net N$3: track 35.6 -> 0.00 mm
- net N$6: track 34.4 -> 0.00 mm
- net N$2: track 25.6 -> 0.00 mm
- net N$7: track 24.3 -> 0.00 mm
- net N$8: track 16.9 -> 0.00 mm
Other:
- board size 113.2 x 113 mm -> 86 x 83 mm
- board text added: "0.093" thick Lexan"
- board text added: "1/16" thick aluminum angle"
- board text added: "Battery Mart Part #: SLA-12V14-F2 battery width: 152mm hole spacing on bottom of box: 166mm"
- board text added: "front edge of box"
- board text removed: "Box center line"
- board text removed: "Gnd Vcc Out En"
- board text removed: "Lighting UPS Sensor V1.1 June 2017"
- board text removed: "Motion Detector"
- board text removed: "Photocell"
- board text removed: "The corresponding holes in the box are to be located 17.5mm down from the top edge"
