File: LightingUPSEagle/LightingUPS-Sensor_v1-1.brd (EAGLE design)
At the start: 84 x 36 mm, 5 parts

Commit message: Add files via upload
Parts:
- moved U$1 1.00 mm to (24.0, 9.53)
Changed lines of the file:
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@@
 <elements>
 <element name="U$5" library="special-drill" package="DRILL_0.2500" value="" x="8.89" y="18"/>
-<element name="U$1" library="special-drill" package="DRILL_0.2500" value="" x="23" y="9.525"/>
+<element name="U$1" library="special-drill" package="DRILL_0.2500" value="" x="24" y="9.525"/>
 <element name="R1" library="SparkFun-Sensors" package="PHOTOCELL" value="PHOTOCELLPTH" x="77" y="18" smashed="yes" rot="R270">
 <attribute name="NAME" x="73.4" y="21" size="0.8128" layer="25" rot="R270"/>
